File: Ponderada/Ponderada.kicad_pcb (KiCad board)
At the start: 2 copper layers, 8 parts, among them J1 Conn_01x02_Pin, K1 Relay_SPDT, Q1 BC548, U1 Pico, U2 LM35-LP

Commit message: update
Parts:
- moved J1 55.5 mm to (207.0, 129.0)
- moved U2 29.0 mm to (182.3, 107.4)
- moved K1 22.4 mm to (185.2, 123.8)
- moved D1 15.0 mm to (171.5, 116.0)
- moved R2 11.2 mm to (138.3, 115.5)
- moved R1 10.0 mm to (137.8, 121.5)
- moved U1 9.51 mm to (122.1, 111.8)
- moved Q1 7.49 mm to (173.6, 124.4), turned to 90 degrees
Connections:
- D1 pad 2: unconnected-(D1-A-Pad2) -> GND
Routing:
- net Analogico: track 0.00 -> 49.3 mm
- net VCC: track 0.00 -> 35.5 mm
- net GND: track 0.00 -> 18.1 mm
- net Net-(Q1-C): track 0.00 -> 14.9 mm
- net Net-(J1-Pin_2): track 0.00 -> 13.4 mm
- net Net-(Q1-B): track 0.00 -> 11.1 mm
- net Net-(D1-K): track 0.00 -> 7.97 mm
- net GP22: track 0.00 -> 7.39 mm
- net GP21: track 0.00 -> 7.15 mm
- net Net-(J1-Pin_1): track 0.00 -> 5.30 mm
- added copper zone on F.Cu, net (none)
